Commit message: lidar girat

File: src/rubot_mecanum_description/urdf/rubot_rp.urdf (robot description, URDF)
Before this commit: robot nexus, 8 links, 7 joints
Links:
- link camera: geometry collision box size=0.075 0.075 0.025; visual mesh filename=package://rubot_mecanum_description/meshes/nexus/piCamera.s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 scale=0.0025 0.0025 0.0025
- link upper_left_wheel: geometry collision cylinder length=0.0505 radius=0.05; visual mesh filename=package://rubot_mecanum_description/meshes/nexus/mecanum_wh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 scale=0.001 0.001 0.001
Joints:
- joint joint_camera: axis 0 1 0 -> 0 0 1; origin xyz=0.236 0.076 0.072 rpy=0 0 0 -> xyz=0.16 0 0.05 rpy=0 0 0
- joint lower_left_wheel_joint: origin xyz=0 0 0 rpy=0 0 0 -> xyz=0 0.042 0 rpy=0 0 0; parent base_link -> lower_left_wheel_shaft

Commit message: message

File: src/rubot_mecanum_description/urdf/rubot_rp.urdf (robot description, URDF)
Before this commit: robot nexus, 8 links, 7 joints
Joints:
- joint scan_joint: origin xyz=0.111 0.076 0.124 rpy=0 0 0 -> xyz=0 0 0.124 rpy=0 0 3.14

Commit message: message

File: src/rubot_mecanum_description/urdf/rubot_rp.urdf (robot description, URDF)
Before this commit: robot nexus, 8 links, 7 joints
Links:
- link base_scan: geometry collision cylinder length=0.01575 radius=0.0275; visual mesh filename=package://rubot_mecanum_description/meshes/nexus/X4.stl scale=0.0015 0.0015 0.0015
Joints:
- joint scan_joint: origin xyz=0 0 0.124 rpy=0 0 3.14 -> xyz=0 0.1 0.09 rpy=0 0 3.14

Commit message: message

File: src/rubot_mecanum_description/urdf/rubot_rp.urdf (robot description, URDF)
Before this commit: robot nexus, 8 links, 7 joints
Links:
- link base_scan: geometry collision cylinder length=0.01575 radius=0.0275; visual mesh filename=package://rubot_mecanum_description/meshes/rubot/lidar.stl scale=0.001 0.001 0.001
Joints:
- joint scan_joint: origin xyz=0 0.1 0.09 rpy=0 0 3.14 -> xyz=0.111 0.076 0.124 rpy=0 0 3.14
